Commit message: launch files added

File: src/try1/urdf/filev3.xacro (robot description, xacro)
@@ -55,8 +55,8 @@
     </visual>
   </link>-->
-<joint name="one" type="continuous">
+<!--<joint name="one" type="continuous">
 <parent link="base"/>
 <child link="laser_vert_bottom"/>
-</joint>
+</joint>-->
 <!--<joint name="two" type="continuous">
 <parent link="base"/>

Commit message: Updated axis

File: src/try1/urdf/filev3.xacro (robot description, xacro)
@@ -85,4 +85,6 @@
 <parent link="base"/>
 <child link="wheel_center"/>
+<limit effort="30" velocity="1"/>
+<axis xyz="0 0 1"/>
 </joint>
 <!--</xacro:macro>
@@ -115,4 +117,6 @@
 <parent link="base"/>
 <child link="wheel_${suffix}"/>
+<limit effort="30" velocity="1"/>
+<axis xyz="0 0 1"/>
 </joint>
 </xacro:macro>

File: src/try1/urdf/new.urdf (robot description, URDF)
Before this commit: robot amazingRobot, 9 links, 9 joints
Joints:
- removed joint one
- joint five_left: axis (none) -> 0 1 0; limit (none) -> effort=30 velocity=1
- joint five_right: axis (none) -> 0 1 0; limit (none) -> effort=30 velocity=1
- joint six: axis (none) -> 0 1 0; limit (none) -> effort=30 velocity=1
